File: elektronik/lüfterklappenelektronik.sch (KiCad schematic (older format))
At the start: 44 parts, among them P101 CONN_01X04, P102 FAN_230VAC_Phase, P103 PressureSensor3, P104 PressureSensor1, P105 PressureSensor2, P106 DamperMotor1, P107 DamperMotor2, P108 DamperMotor3, P109 CONN_01X03, Q101 IRF9540N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

Commit message: esp32 start
Parts:
- removed U?: WeMos_mini, symbol ESP8266wemosD1:WeMos_mini
- added C? (x3): 22uF/10V, symbol Device:C
- added C? (x2): 0.1uF/50V, symbol Device:C
- added D?: LED, symbol Device:LED
- added P?: USB_C_Plug_USB2.0, symbol Connector:USB_C_Plug_USB2.0
- added R?: 2K, symbol Device:R
- added R?: 10K(5%), symbol Device:R
- added U?: ESP32-WROOM-32E, RF_Module:ESP32-WROOM-32, symbol RF_Module:ESP32-WROOM-32D
- added U?: AMS1117-3.3, Package_TO_SOT_SMD:SOT-223-3_TabPin2, symbol Regulator_Linear:AMS1117-3.3
Connections:
- net labels added: +3V3, ESP_EN
- wire segments 94 -> 110

Commit message: esp32 schaltung
Parts:
- removed A?: Arduino_Nano_v3.x, Module:Arduino_Nano, symbol MCU_Module:Arduino_Nano_v3.x
- removed P?: USB_C_Plug_USB2.0, symbol Connector:USB_C_Plug_USB2.0
- added C?: 4.7µF/6.3V(10%), symbol Device:C
- added C?: 0.1µF/50V(10%), symbol Device:C
- added C? (x2): 0.1µF/50V, symbol Device:C
- added D?: BAT760-7, Diode_THT:D_DO-35_SOD27_P7.62mm_Horizontal, symbol Diode:BAT85
- added D? (x3): LESD5D5.0CT1G, symbol Device:D_TVS_ALT
- added J?: USB_B_Micro, FootprintsTittelbach:USB_Micro-B_C77238, symbol Connector:USB_B_Micro
- added J?: LAN Breakout Connector, Connector_PinSocket_2.54mm:PinSocket_1x08_P2.54mm_Vertical_SMD_Pin1Left, symbol Connector:Conn_01x08_Female
- added Q? (x2): Q_NPN_Darlington_BEC, Package_TO_SOT_SMD:SOT-23, symbol Device:Q_NPN_Darlington_BEC
- added R?: 22.1K(5%), symbol Device:R
- added R?: 47.5K(5%), symbol Device:R
- added R? (x3): 10K(5%), symbol Device:R
- added R?: 2K(5%), symbol Device:R
- added R? (x2): 0R(5%), symbol Device:R
- added SW? (x2): SW_Push, Button_Switch_SMD:SW_SPST_B3SL-1022P, symbol Switch:SW_Push
- added U?: CP2102N-A01-GQFN28, Package_DFN_QFN:QFN-28-1EP_5x5mm_P0.5mm_EP3.35x3.35mm, symbol Interface_USB:CP2102N-A01-GQFN28
- Q101: value IRF9540N -> IRLR8743TRPBF; Distributor (none) -> LCSC; LCSCPartN (none) -> C51360; MF (none) -> Infineon Technologies; MP (none) -> IRLR8743TRPBF
- Q102, Q103: value IRF9540N -> IRLR8743TRPBF
- U?: Distributor (none) -> LCSC; LCSCPartN (none) -> C701343; MF (none) -> Espressif Systems; MP (none) -> ESP32-WROOM-32E(16MB)
- U?: footprint Package_TO_SOT_SMD:SOT-223-3_TabPin2 -> Package_TO_SOT_SMD:SOT-89-3; Distributor (none) -> LCSC; LCSCPartN (none) -> C347256; MF (none) -> UMW(Youtai Semiconductor Co., Ltd.); MP (none) -> AMS1117-3.3
Connections:
- net labels added: +VDC, CTS, DCD, DSR, DTR, IO0, RI, RTS, RXD, RXD0, TXD, TXD0, USB_D+, USB_D-, VBUS
- wire segments 110 -> 198
- no-connect marks 12 -> 27
Other:
- note added: "30V Reverse Protection"
- moved on the sheet: U?

Commit message: nice looking schematic
Parts:
- removed C?: 100nF, symbol Device:C
- removed J?: LAN Breakout Connector, Connector_PinSocket_2.54mm:PinSocket_1x08_P2.54mm_Vertical_SMD_Pin1Left, symbol Connector:Conn_01x08_Female
- removed P109: CONN_01X03, Pin_Headers:Pin_Header_Straight_1x03, symbol lüfterklappenelektronik-rescue:CONN_01X03
- added D? (x8): LESD5D5.0CT1G, symbol Device:D_TVS_ALT
- added D?: GREEN_LED, LED_SMD:LED_0603_1608Metric, symbol Device:LED
- added J?: Conn_01x05_Male, symbol Connector:Conn_01x05_Male
- added J?: Conn_FAN, symbol Connector:Conn_01x02_Female
- added J?: Conn_LAN_ENC28J60, symbol Connector_Generic:Conn_02x05_Odd_Even
- added R?: 110(1%), symbol Device:R
- added R? (x8): 22(1%), symbol Device:R
- C101, P102, R108, U104, VR101: DNF (none) -> DNF
- R101, R102, R103: value #120 -> 43(1%)
- R104, R105, R106: value #2K2 -> 2K2
- R107: value 100 -> 160(1%)
- R?: value 0 -> 22(1%)
- U101, U103: value #Gabellichtschranke -> Gabellichtschranke
- U102: value #Gabellichtschranke -> Gabellichtschranke; DNF (none) -> DNF
Connections:
- net labels added: LAN_CLKOUT, LAN_CS, LAN_INT, LAN_RESET, LAN_WOL, ONBOARD_LED, PS1_CS, PS2_CS, PS3_CS, SCL, SDA, UCD+, UCD-
- net labels removed: PS1SS, PS2SS, PS3SS, RX, TX
- wire segments 198 -> 234
- no-connect marks 27 -> 32
Other:
- note added: "11mA over 160R\nasuming 1.5V IRLED"
- note added: "37..42mA"
- note added: "Power Budget:\n0120mA ... Gabellichtschranken\n1500mA ... ESP32\n0010mA ... Green LED\n0011mA ... IR Led inside FAN SSR"
- note added: "mirrored connector so ENC28J60 boards can directly connected"
- moved on the sheet: C101, C?, D101, D102, D103, D?, J?, P101, P102, P103, P104, P105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

Commit message: selected all footprints and components
Parts:
- removed C? (x2): 100nF, symbol Device:C
- removed C?: 1000µF, symbol Device:CP
- removed C? (x2): 22uF/10V, symbol Device:C
- removed C?: 0.1uF/50V, symbol Device:C
- removed C?: 0.1µF/50V(10%), symbol Device:C
- removed C? (x2): 0.1µF/50V, symbol Device:C
- removed D? (x3): D_Small, symbol Device:D_Small
- removed D?: LED, symbol Device:LED
- added C102, C104, C107, C108, C109, C115: 100nF/50V, Capacitor_SMD:C_0603_1608Metric, symbol Device:C
- added C103: 220µF/6.3V(20%), Capacitor_SMD:C_1206_3216Metric, symbol Device:C
- added C111, C112: 22uF/25V(10%), Capacitor_SMD:C_1210_3225Metric, symbol Device:C
- added D106, D107, D108: BAT760-7, Diode_THT:D_DO-35_SOD27_P7.62mm_Horizontal, symbol Diode:BAT85
- added D113: GREEN_LED, LED_SMD:LED_0603_1608Metric, symbol Device:LED
- added JP101: Jumper µC Supply, Connector_PinHeader_2.54mm:PinHeader_1x03_P2.54mm_Vertical, symbol Device:Jumper_NC_Dual
- added P109: PWR_BUS_CONN2, TerminalBlock_RND:TerminalBlock_RND_205-00289_1x04_P5.08mm_Horizontal, symbol lüfterklappenelektronik-rescue:CONN_01X04
- C101: value C_SSR -> #C_SSR
- C105: renamed from C?; value 1µF -> 1µF/50V; footprint (none) -> Capacitor_SMD:C_0603_1608Metric; Distributor (none) -> LCSC; LCSCPartN (none) -> C105174; MF (none) -> Taiyo Yuden; MP (none) -> UMK107AB7105KA-T
- C106: renamed from C?; value 10µF -> 10µF/25V; footprint (none) -> Capacitor_SMD:C_0805_2012Metric; Distributor (none) -> LCSC; LCSCPartN (none) -> C40894; MF (none) -> FH; MP (none) -> 0805X106K250NT
- C110: renamed from C?; value 22uF/10V -> 22uF/25V(10%); footprint (none) -> Capacitor_SMD:C_1210_3225Metric; Distributor (none) -> LCSC; LCSCPartN (none) -> C337455; MF (none) -> Taiyo Yuden; MP (none) -> TMK325B7226KM-TR
- C113: renamed from C?; value 0.1uF/50V -> 100nF/50V; footprint (none) -> Capacitor_SMD:C_0603_1608Metric; Distributor (none) -> LCSC; LCSCPartN (none) -> C42998; MF (none) -> FH; MP (none) -> 0603F104M500NT
- C114: renamed from C?; footprint (none) -> Capacitors_SMD:C_0603
- D101, D102, D103: footprint (none) -> Diode_SMD:D_SMB; Distributor (none) -> LCSC; LCSCPartN (none) -> C353175; MF (none) -> Shandong Jingdao Microelectronics; MP (none) -> SS54B
- D104, D109, D110, D111, D112, D114, D116, D117, D118, D119, D120: renamed from D?; footprint (none) -> Diode_SMD:D_SOD-523
- J101: renamed from J?; footprint (none) -> Connector_PinHeader_2.54mm:PinHeader_1x05_P2.54mm_Vertical; DNF (none) -> DNF
- J102: renamed from J?; footprint (none) -> Connector_JST:JST_XH_B2B-XH-A_1x02_P2.50mm_Vertical
- J103: renamed from J?; footprint (none) -> Connector_PinSocket_2.54mm:PinSocket_2x05_P2.54mm_Vertical_SMD
- P101: value CONN_01X04 -> PWR_BUS_CONN1; footprint Terminal_Blocks:TerminalBlock_Pheonix_MPT-2.54mm_4pol -> TerminalBlock_RND:TerminalBlock_RND_205-00289_1x04_P5.08mm_Horizontal; Distributor (none) -> LCSC; LCSCPartN (none) -> C8446; MF (none) -> Ningbo Kangnex Elec; MP (none) -> WJ2EDGRC-5.08-4P
- P102: value FAN_230VAC_Phase -> #FAN_230VAC_Phase
- R108: value R_SSR -> #R_SSR
- R109, R110, R111: value 100 -> 100(1%); footprint Resistors_ThroughHole:Resistor_Horizontal_RM7mm -> Resistors_SMD:R_0603
- R112, R113, R114, R115, R116, R117, R118, R119, R120, R121, R122, R123, R124, R125, R126, R127, R128, R129, R130, R131: renamed from R?; footprint (none) -> Resistor_SMD:R_0603_1608Metric
- U104: value ZG3NC-240B -> #ZG3NC-240B; footprint Pin_Headers:Pin_Header_Straight_1x02 -> (none)
- VR101: value S7K275 -> #S7K275
- gave numbers to parts that had none: 10
Connections:
- net +12V: now also P101.1 (P1), JP101.1, P109.4 (P4); no longer C110.1, D115.1 (K), P101.4 (P4), R125.1, U106.3 (VI)
- net +3V3: now also C103.1, C104.1, C107.1, C111.1, C112.1, C115.1
- net +5V: now also P101.3 (P3), JP101.3, P109.2 (P2)
- net ESP_EN: now also C102.1, C108.1
- net EndstopDamper1: now also U105.28 (IO17), D106.2 (A); no longer U101.3 (Rh)
- net EndstopDamper2: now also U105.30 (IO18), D107.2 (A); no longer U102.3 (Rh)
- net EndstopDamper3: now also U105.31 (IO19), D108.2 (A); no longer U103.3 (Rh)
- net GND: now also P101.4 (P4), C102.2, C103.2, C104.2, C107.2, C108.2, C109.2, C111.2, C112.2, C115.2, D113.1 (K), P109.1 (P1); no longer P101.1 (P1)
- net IO0: now also C109.1
- net PJON: now also P101.2 (P2), P109.3 (P3); no longer P101.3 (P3)
- net at R125.2: now also D113.2 (A)
- new net: D106.1 (K), U101.3 (Rh)
- new net: D107.1 (K), U102.3 (Rh)
- new net: D108.1 (K), U103.3 (Rh)
- new net +VDC: C110.1, D115.1 (K), JP101.2, R125.1, U106.3 (VI)
- no-connect marks 32 -> 31
Other:
- note added: "30V Reverse Protection\nprotecting USB from 12V"
- note added: "PWM possible for Damper Pins"
- note added: "Power Use:\n0120mA ... Gabellichtschranken\n1000mA ... ESP32\n0010mA ... Green LED\n0011mA ... IR Led inside FAN SSR"
- note added: "Widerstände schon auf Gabellichtschranke???"
- note removed: "30V Reverse Protection"
- note removed: "Power Budget:\n0120mA ... Gabellichtschranken\n1500mA ... ESP32\n0010mA ... Green LED\n0011mA ... IR Led inside FAN SSR"
- moved on the sheet: P101

Commit message: update footprint
Parts:
- added J105: #Stecker, symbol Connector:Conn_01x02_Male
- J102: footprint Connector_JST:JST_XH_B2B-XH-A_1x02_P2.50mm_Vertical -> Connect:PINHEAD1-2; Distributor (none) -> LCSC; LCSCPartN (none) -> C30436; MF (none) -> BOOMELE(Boom Precision Elec); MP (none) -> C30436
- U101, U103: footprint Pin_Headers:Pin_Header_Straight_1x04 -> FootprintsTittelbach:Ckmtw_2510S-4P; Distributor (none) -> LCSC; LCSCPartN (none) -> C140769; MF (none) -> Ckmtw(Shenzhen Cankemeng); MP (none) -> 2510S-4P
- U102: footprint Pin_Headers:Pin_Header_Straight_1x04 -> FootprintsTittelbach:Ckmtw_2510S-4P; DNF DNF -> (none); Distributor (none) -> LCSC; LCSCPartN (none) -> C140769; MF (none) -> Ckmtw(Shenzhen Cankemeng); MP (none) -> 2510S-4P
Connections:
- net +3V3: no longer U104.3
- net at D104.1 (A1), J102.2 (Pin_2), R107.1: no longer U104.4
- new net: J105.1 (Pin_1), U104.3
- new net: J105.2 (Pin_2), U104.4
Other:
- note added: "Not part of PCB"
Changed lines of the file:
@@
 F 0 "U101" H 1750 2125 50  0000 C CNN
 F 1 "Gabellichtschranke" H 1750 2034 50  0000 C CNN
-F 2 "Pin_Headers:Pin_Header_Straight_1x04" H 1750 1700 50  0000 C CNN
-F 3 "" H 1750 1700 50  0000 C CNN
-F 4 "" H 1750 1700 50  0001 C CNN "DNF"
+F 2 "FootprintsTittelbach:Ckmtw_2510S-4P" H 1750 1700 50  0001 C CNN
+F 3 "https://datasheet.lcsc.com/szlcsc/1811061121_BOOMELE-Boom-Precision-Elec-C31753_C31753.pdf" H 1750 1700 50  0001 C CNN
+F 4 "Ckmtw(Shenzhen Cankemeng)" H 1750 1700 50  0001 C CNN "MF"
+F 5 "2510S-4P" H 1750 1700 50  0001 C CNN "MP"
+F 6 "LCSC" H 1750 1700 50  0001 C CNN "Distributor"
+F 7 "C140769" H 1750 1700 50  0001 C CNN "LCSCPartN"
 	1    1750 1700
 	1    0    0    -1
@@
 EndstopDamper1
 $Comp
-L lüfterklappenelektronik-rescue:PHOTORESISTOR U102
-U 1 1 5741D5DE
-P 1750 3450
-F 0 "U102" H 1750 3875 50  0000 C CNN
-F 1 "Gabellichtschranke" H 1750 3784 50  0000 C CNN
-F 2 "Pin_Headers:Pin_Header_Straight_1x04" H 1750 3450 50  0000 C CNN
-F 3 "" H 1750 3450 50  0000 C CNN
-F 4 "DNF" H 1750 3450 50  0001 C CNN "DNF"
-	1    1750 3450
-	1    0    0    -1
-$EndComp
-$Comp
 L lüfterklappenelektronik-rescue:R R102
 U 1 1 5741D5E4
@@
 Text Label 2650 3250 0    60   ~ 0
 EndstopDamper2
-$Comp
-L lüfterklappenelektronik-rescue:PHOTORESISTOR U103
-U 1 1 5741D70C
-P 1750 5100
-F 0 "U103" H 1750 5525 50  0000 C CNN
-F 1 "Gabellichtschranke" H 1750 5434 50  0000 C CNN
-F 2 "Pin_Headers:Pin_Header_Straight_1x04" H 1750 5100 50  0000 C CNN
-F 3 "" H 1750 5100 50  0000 C CNN
-	1    1750 5100
-	1    0    0    -1
-$EndComp
 $Comp
 L lüfterklappenelektronik-rescue:R R103
@@
 	1    0    0    -1
 $EndComp
-Wire Wire Line
-	3850 6200 3850 6550
 $Comp
 L Connector:Conn_01x02_Female J102
 U 1 1 5FB1F52D
 P 4050 6650
-F 0 "J102" H 4078 6626 50  0000 L CNN
+F 0 "J102" H 3950 6750 50  0000 L CNN
 F 1 "Conn_FAN" H 3700 6450 50  0000 L CNN
-F 2 "Connector_JST:JST_XH_B2B-XH-A_1x02_P2.50mm_Vertical" H 4050 6650 50  0001 C CNN
+F 2 "Connect:PINHEAD1-2" H 4050 6650 50  0001 C CNN
 F 3 "~" H 4050 6650 50  0001 C CNN
+F 4 " BOOMELE(Boom Precision Elec) " H 4050 6650 50  0001 C CNN "MF"
+F 5 "C30436" H 4050 6650 50  0001 C CNN "MP"
+F 6 "LCSC" H 4050 6650 50  0001 C CNN "Distributor"
+F 7 "C30436" H 4050 6650 50  0001 C CNN "LCSCPartN"
 	1    4050 6650
 	1    0    0    -1
 $EndComp
-Wire Wire Line
-	4400 6600 4400 6550
-Wire Wire Line
-	4400 6550 3850 6550
-Wire Wire Line
-	4400 6600 4650 6600
-Connection ~ 3850 6550
-Wire Wire Line
-	3850 6550 3850 6650
-Wire Wire Line
-	3850 6750 3850 6800
-Wire Wire Line
-	3850 6800 4650 6800
-Connection ~ 3850 6750
 $Comp
 L power:+3V3 #PWR0120
@@
 	1    0    0    -1
 $EndComp
+$Comp
+L Connector:Conn_01x02_Male J105
+U 1 1 60ECC0FE
+P 4250 6650
+F 0 "J105" H 4358 6831 50  0000 C CNN
+F 1 "#Stecker" H 4358 6740 50  0000 C CNN
+F 2 "" H 4250 6650 50  0001 C CNN
+F 3 "~" H 4250 6650 50  0001 C CNN
+F 4 "DNF" H 4250 6650 50  0001 C CNN "DNF"
+	1    4250 6650
+	1    0    0    -1
+$EndComp
+Wire Wire Line
+	3850 6200 3850 6650
+Wire Wire Line
+	4650 6600 4650 6650
+Wire Wire Line
+	4450 6650 4650 6650
+Wire Wire Line
+	4450 6750 4650 6750
+Wire Wire Line
+	4650 6750 4650 6800
+Wire Notes Line
+	4200 6250 6850 6250
+Wire Notes Line
+	6850 6250 6850 7350
+Wire Notes Line
+	6850 7350 4200 7350
+Wire Notes Line
+	4200 7350 4200 6250
+Text Notes 4250 7300 0    50   ~ 0
+Not part of PCB
+$Comp
+L lüfterklappenelektronik-rescue:PHOTORESISTOR U102
+U 1 1 60F4914E
+P 1750 3450
+F 0 "U102" H 1750 3875 50  0000 C CNN
+F 1 "Gabellichtschranke" H 1750 3784 50  0000 C CNN
+F 2 "FootprintsTittelbach:Ckmtw_2510S-4P" H 1750 3450 50  0001 C CNN
+F 3 "https://datasheet.lcsc.com/szlcsc/1811061121_BOOMELE-Boom-Precision-Elec-C31753_C31753.pdf" H 1750 3450 50  0001 C CNN
+F 4 "Ckmtw(Shenzhen Cankemeng)" H 1750 3450 50  0001 C CNN "MF"
+F 5 "2510S-4P" H 1750 3450 50  0001 C CNN "MP"
+F 6 "LCSC" H 1750 3450 50  0001 C CNN "Distributor"
+F 7 "C140769" H 1750 3450 50  0001 C CNN "LCSCPartN"
+	1    1750 3450
+	1    0    0    -1
+$EndComp
+$Comp
+L lüfterklappenelektronik-rescue:PHOTORESISTOR U103
+U 1 1 60F49E0C
+P 1750 5100
+F 0 "U103" H 1750 5525 50  0000 C CNN
+F 1 "Gabellichtschranke" H 1750 5434 50  0000 C CNN
+F 2 "FootprintsTittelbach:Ckmtw_2510S-4P" H 1750 5100 50  0001 C CNN
+F 3 "https://datasheet.lcsc.com/szlcsc/1811061121_BOOMELE-Boom-Precision-Elec-C31753_C31753.pdf" H 1750 5100 50  0001 C CNN
+F 4 "Ckmtw(Shenzhen Cankemeng)" H 1750 5100 50  0001 C CNN "MF"
+F 5 "2510S-4P" H 1750 5100 50  0001 C CNN "MP"
+F 6 "LCSC" H 1750 5100 50  0001 C CNN "Distributor"
+F 7 "C140769" H 1750 5100 50  0001 C CNN "LCSCPartN"
+	1    1750 5100
+	1    0    0    -1
+$EndComp
