File: elektronik/lüfterklappenelektronik.sch (KiCad schematic (older format))
At the start: 121 parts, among them J101 Conn_01x05_Male, J102 Ckmtw_2510S-2P, J103 Conn_LAN_ENC28J60, J104 USB_B_Micro, J105 #Stecker, J106 WJ2EDGRC-5.08-2P, J107 WJ2EDGRC-5.08-2P, J108 WJ2EDGRC-5.08-2P, P101 PWR_BUS_CONN1, P102 #FAN_230VAC_Phase, P103 PressureSensor3, P104 PressureSensor1, P105 PressureSensor2, P109 PWR_BUS_CONN2, Q101 IRLR8743TRPBF, Q102 IRLR8743TRPBF, Q103 IRLR8743TRPBF, Q104 Q_NPN_Darlington_BEC, Q105 Q_NPN_Darlington_BEC, SW101 SW_Push, SW102 SW_Push, U101 Gabellichtschranke, U102 Gabellichtschranke, U103 Gabellichtschranke, U104 #ZG3NC-240B, U105 ESP32-WROOM-32E, U106 AMS1117-3.3, U107 CP2102N-A01-GQFN28

Commit message: fixes. One fuckup remaining: damper2 needs different connector now
Parts:
- C111, D101, D109, D115, J103, J104, L107, Q104, Q105, R118, R122, R125, SW101, U105, U106, U107: Type (none) -> SMT
- D105: Field7 C264449 -> (none); LCSCPartN (none) -> C264449
- D113: Field7 C264449 -> (none); LCSCPartN (none) -> C264449; Type (none) -> SMT
- J101, J102, JP101, P101, P109, U101, U102, U103: Type (none) -> TH
- P103, P104, P105: footprint Pin_Headers:Pin_Header_Straight_1x06 -> Connector_PinHeader_2.54mm:PinHeader_1x06_P2.54mm_Vertical; DNF (none) -> DNF; Type (none) -> TH
Changed lines of the file:
@@
 F 6 "LCSC" V 5150 1300 50  0001 C CNN "Distributor"
 F 7 "C353175" V 5150 1300 50  0001 C CNN "LCSCPartN"
+F 8 "SMT" V 5150 1300 50  0001 C CNN "Type"
 	1    5150 1300
 	0    1    1    0
@@
 F 6 "LCSC" H 1600 1700 50  0001 C CNN "Distributor"
 F 7 "C140769" H 1600 1700 50  0001 C CNN "LCSCPartN"
+F 8 "TH" H 1600 1700 50  0001 C CNN "Type"
 	1    1600 1700
 	1    0    0    -1
@@
 F 0 "P103" H 2027 8941 50  0000 L CNN
 F 1 "PressureSensor3" H 2027 8850 50  0000 L CNN
-F 2 "Pin_Headers:Pin_Header_Straight_1x06" H 1950 8900 50  0001 C CNN
+F 2 "Connector_PinHeader_2.54mm:PinHeader_1x06_P2.54mm_Vertical" H 1950 8900 50  0001 C CNN
 F 3 "" H 1950 8900 50  0000 C CNN
+F 4 "DNF" H 1950 8900 50  0001 C CNN "DNF"
+F 5 "TH" H 1950 8900 50  0001 C CNN "Type"
 	1    1950 8900
 	1    0    0    -1
@@
 F 0 "P105" H 2027 7841 50  0000 L CNN
 F 1 "PressureSensor2" H 2027 7750 50  0000 L CNN
-F 2 "Pin_Headers:Pin_Header_Straight_1x06" H 1950 7800 50  0001 C CNN
+F 2 "Connector_PinHeader_2.54mm:PinHeader_1x06_P2.54mm_Vertical" H 1950 7800 50  0001 C CNN
 F 3 "" H 1950 7800 50  0000 C CNN
+F 4 "DNF" H 1950 7800 50  0001 C CNN "DNF"
+F 5 "TH" H 1950 7800 50  0001 C CNN "Type"
 	1    1950 7800
 	1    0    0    -1
@@
 F 0 "P104" H 2027 6691 50  0000 L CNN
 F 1 "PressureSensor1" H 2027 6600 50  0000 L CNN
-F 2 "Pin_Headers:Pin_Header_Straight_1x06" H 1950 6650 50  0001 C CNN
+F 2 "Connector_PinHeader_2.54mm:PinHeader_1x06_P2.54mm_Vertical" H 1950 6650 50  0001 C CNN
 F 3 "" H 1950 6650 50  0000 C CNN
+F 4 "TH" H 1950 6650 50  0001 C CNN "Type"
+F 5 "DNF" H 1950 6650 50  0001 C CNN "DNF"
 	1    1950 6650
 	1    0    0    -1
@@
 F 2 "Resistor_SMD:R_0603_1608Metric" V 8930 6250 50  0001 C CNN
 F 3 "~" H 9000 6250 50  0001 C CNN
+F 4 "SMT" V 9000 6250 50  0001 C CNN "Type"
 	1    9000 6250
 	0    -1   1    0
@@
 F 6 "LCSC" H 8050 5750 50  0001 C CNN "Distributor"
 F 7 "C701343" H 8050 5750 50  0001 C CNN "LCSCPartN"
+F 8 "SMT" H 8050 5750 50  0001 C CNN "Type"
 	1    8050 5750
 	1    0    0    -1
@@
 F 6 "LCSC" H 12850 1850 50  0001 C CNN "Distributor"
 F 7 "C347256" H 12850 1850 50  0001 C CNN "LCSCPartN"
+F 8 "SMT" H 12850 1850 50  0001 C CNN "Type"
 	1    12850 1850
 	1    0    0    -1
@@
 F 2 "Resistor_SMD:R_0603_1608Metric" V 11330 2000 50  0001 C CNN
 F 3 "~" H 11400 2000 50  0001 C CNN
+F 4 "SMT" H 11400 2000 50  0001 C CNN "Type"
 	1    11400 2000
 	1    0    0    -1
@@
 F 6 "LCSC" H 11600 3700 50  0001 C CNN "Distributor"
 F 7 "C124187" H 11600 3700 50  0001 C CNN "LCSCPartN"
+F 8 "SMT" H 11600 3700 50  0001 C CNN "Type"
 	1    11600 3700
 	-1   0    0    1
@@
 F 6 "LCSC" H 13500 3900 50  0001 C CNN "Distributor"
 F 7 "C77238" H 13500 3900 50  0001 C CNN "LCSCPartN"
+F 8 "SMT" H 13500 3900 50  0001 C CNN "Type"
 	1    13500 3900
 	1    0    0    -1
@@
 F 6 "LCSC" H 14250 8400 50  0001 C CNN "Distributor"
 F 7 "C428937" H 14250 8400 50  0001 C CNN "LCSCPartN"
+F 8 "SMT" H 14250 8400 50  0001 C CNN "Type"
 	1    14250 8400
 	1    0    0    -1
@@
 F 6 "LCSC" H 8450 9600 50  0001 C CNN "Distributor"
 F 7 "C164885" H 8450 9600 50  0001 C CNN "LCSCPartN"
+F 8 "SMT" H 8450 9600 50  0001 C CNN "Type"
 	1    8450 9600
 	1    0    0    -1
@@
 F 6 "LCSC" H 8450 10200 50  0001 C CNN "Distributor"
 F 7 "C164885" H 8450 10200 50  0001 C CNN "LCSCPartN"
+F 8 "SMT" H 8450 10200 50  0001 C CNN "Type"
 	1    8450 10200
 	1    0    0    -1
@@
 F 6 "LCSC" H 10700 9200 50  0001 C CNN "Distributor"
 F 7 "C86708" H 10700 9200 50  0001 C CNN "LCSCPartN"
+F 8 "SMT" H 10700 9200 50  0001 C CNN "Type"
 	1    10700 9200
 	1    0    0    -1
@@
 F 6 "LCSC" H 10250 7000 50  0001 C CNN "Distributor"
 F 7 "C383211" H 10250 7000 50  0001 C CNN "LCSCPartN"
+F 8 "SMT" V 10250 7000 50  0001 C CNN "Type"
 	1    10250 7000
 	0    -1   1    0
@@
 F 3 "~" H 2700 10400 50  0001 C CNN
 F 4 "DNF" H 2700 10400 50  0001 C CNN "DNF"
+F 5 "TH" H 2700 10400 50  0001 C CNN "Type"
 	1    2700 10400
 	-1   0    0    1
@@
 F 6 "LCSC" H 4050 6650 50  0001 C CNN "Distributor"
 F 7 "C30436" H 4050 6650 50  0001 C CNN "LCSCPartN"
+F 8 "TH" H 4050 6650 50  0001 C CNN "Type"
 	1    4050 6650
 	1    0    0    -1
@@
 F 5 "19-21SYGD/S530-E2/TR8" V 3600 8650 50  0001 C CNN "MP"
 F 6 "LCSC" V 3600 8650 50  0001 C CNN "Distributor"
-F 7 "C264449" V 3600 8650 50  0001 C CNN "Field7"
+F 7 "C264449" V 3600 8650 50  0001 C CNN "LCSCPartN"
 	1    3600 8650
 	0    -1   -1   0
@@
 F 2 "Resistor_SMD:R_0603_1608Metric" V 10380 5350 50  0001 C CNN
 F 3 "~" H 10450 5350 50  0001 C CNN
+F 4 "SMT" V 10450 5350 50  0001 C CNN "Type"
 	1    10450 5350
 	0    1    1    0
@@
 F 2 "Connector_PinHeader_2.54mm:PinHeader_1x03_P2.54mm_Vertical" H 10150 1500 50  0001 C CNN
 F 3 "~" H 10150 1500 50  0001 C CNN
+F 4 "TH" H 10150 1500 50  0001 C CNN "Type"
 	1    10150 1500
 	-1   0    0    1
@@
 F 6 "LCSC" H 10650 3300 50  0001 C CNN "Distributor"
 F 7 "C8446" H 10650 3300 50  0001 C CNN "LCSCPartN"
+F 8 "TH" H 10650 3300 50  0001 C CNN "Type"
 	1    10650 3300
 	1    0    0    1
@@
 F 6 "LCSC" H 13550 2000 50  0001 C CNN "Distributor"
 F 7 "C337455" H 13550 2000 50  0001 C CNN "LCSCPartN"
+F 8 "SMT" H 13550 2000 50  0001 C CNN "Type"
 	1    13550 2000
 	1    0    0    -1
@@
 F 5 "19-21SYGD/S530-E2/TR8" V 11400 2450 50  0001 C CNN "MP"
 F 6 "LCSC" V 11400 2450 50  0001 C CNN "Distributor"
-F 7 "C264449" V 11400 2450 50  0001 C CNN "Field7"
+F 7 "C264449" V 11400 2450 50  0001 C CNN "LCSCPartN"
+F 8 "SMT" V 11400 2450 50  0001 C CNN "Type"
 	1    11400 2450
 	0    -1   -1   0
@@
 F 6 "LCSC" H 1600 3450 50  0001 C CNN "Distributor"
 F 7 "C140769" H 1600 3450 50  0001 C CNN "LCSCPartN"
+F 8 "TH" H 1600 3450 50  0001 C CNN "Type"
 	1    1600 3450
 	1    0    0    -1
@@
 F 6 "LCSC" H 1600 5100 50  0001 C CNN "Distributor"
 F 7 "C140769" H 1600 5100 50  0001 C CNN "LCSCPartN"
+F 8 "TH" H 1600 5100 50  0001 C CNN "Type"
 	1    1600 5100
 	1    0    0    -1
@@
 F 2 "Connector_PinSocket_2.54mm:PinSocket_2x05_P2.54mm_Vertical_SMD" H 4650 10400 50  0001 C CNN
 F 3 "~" H 4650 10400 50  0001 C CNN
+F 4 "SMT" H 4650 10400 50  0001 C CNN "Type"
 	1    4650 10400
 	1    0    0    -1
@@
 F 6 "LCSC" H 9450 3300 50  0001 C CNN "Distributor"
 F 7 "C8446" H 9450 3300 50  0001 C CNN "LCSCPartN"
+F 8 "TH" H 9450 3300 50  0001 C CNN "Type"
 	1    9450 3300
 	-1   0    0    -1
@@
 F 7 "C96697" V 1150 6400 50  0001 C CNN "LCSCPartN"
 F 8 "2.2kΩ @ 100MHz 100mA 1 1.2Ω 0603 Ferrite Beads RoHS" V 1150 6400 50  0001 C CNN "Specs"
+F 9 "SMT" V 1150 6400 50  0001 C CNN "Type"
 	1    1150 6400
 	0    1    1    0

Commit message: fixed part, footprint still needs fixing
Parts:
- J106, J107, J108: value WJ2EDGRC-5.08-2P -> WJ2EDGVC-5.08-2P; LCSCPartN C3697 -> C8445; MP WJ2EDGRC-5.08-2P -> WJ2EDGVC-5.08-2P
Changed lines of the file:
@@
 P 5900 1250
 F 0 "J106" H 5800 1350 50  0000 L CNN
-F 1 "WJ2EDGRC-5.08-2P" H 5550 1050 50  0000 L CNN
+F 1 "WJ2EDGVC-5.08-2P" H 5550 1050 50  0000 L CNN
 F 2 "FootprintsTittelbach:WJ2EDGRC-5.08-2P" H 5900 1250 50  0001 C CNN
-F 3 "https://datasheet.lcsc.com/szlcsc/1912251631_Ningbo-Kangnex-Elec-WJ2EDGRC-5-08-2P_C3697.pdf" H 5900 1250 50  0001 C CNN
+F 3 "https://datasheet.lcsc.com/szlcsc/1912251635_Ningbo-Kangnex-Elec-WJ2EDGVC-5-08-2P_C8445.pdf" H 5900 1250 50  0001 C CNN
 F 4 "Ningbo Kangnex Elec" H 5900 1250 50  0001 C CNN "MF"
-F 5 "WJ2EDGRC-5.08-2P" H 5900 1250 50  0001 C CNN "MP"
+F 5 "WJ2EDGVC-5.08-2P" H 5900 1250 50  0001 C CNN "MP"
 F 6 "LCSC" H 5900 1250 50  0001 C CNN "Distributor"
-F 7 "C3697" H 5900 1250 50  0001 C CNN "LCSCPartN"
+F 7 "C8445" H 5900 1250 50  0001 C CNN "LCSCPartN"
 	1    5900 1250
 	1    0    0    -1
@@
 P 5900 2900
 F 0 "J107" H 5800 3000 50  0000 L CNN
-F 1 "WJ2EDGRC-5.08-2P" H 5550 2700 50  0000 L CNN
+F 1 "WJ2EDGVC-5.08-2P" H 5550 2700 50  0000 L CNN
 F 2 "FootprintsTittelbach:WJ2EDGRC-5.08-2P" H 5900 2900 50  0001 C CNN
-F 3 "https://datasheet.lcsc.com/szlcsc/1912251631_Ningbo-Kangnex-Elec-WJ2EDGRC-5-08-2P_C3697.pdf" H 5900 2900 50  0001 C CNN
+F 3 "https://datasheet.lcsc.com/szlcsc/1912251635_Ningbo-Kangnex-Elec-WJ2EDGVC-5-08-2P_C8445.pdf" H 5900 2900 50  0001 C CNN
 F 4 "Ningbo Kangnex Elec" H 5900 2900 50  0001 C CNN "MF"
-F 5 "WJ2EDGRC-5.08-2P" H 5900 2900 50  0001 C CNN "MP"
+F 5 "WJ2EDGVC-5.08-2P" H 5900 2900 50  0001 C CNN "MP"
 F 6 "LCSC" H 5900 2900 50  0001 C CNN "Distributor"
-F 7 "C3697" H 5900 2900 50  0001 C CNN "LCSCPartN"
+F 7 "C8445" H 5900 2900 50  0001 C CNN "LCSCPartN"
 	1    5900 2900
 	1    0    0    -1
@@
 P 5900 4550
 F 0 "J108" H 5800 4650 50  0000 L CNN
-F 1 "WJ2EDGRC-5.08-2P" H 5550 4350 50  0000 L CNN
+F 1 "WJ2EDGVC-5.08-2P" H 5550 4350 50  0000 L CNN
 F 2 "FootprintsTittelbach:WJ2EDGRC-5.08-2P" H 5900 4550 50  0001 C CNN
-F 3 "https://datasheet.lcsc.com/szlcsc/1912251631_Ningbo-Kangnex-Elec-WJ2EDGRC-5-08-2P_C3697.pdf" H 5900 4550 50  0001 C CNN
+F 3 "https://datasheet.lcsc.com/szlcsc/1912251635_Ningbo-Kangnex-Elec-WJ2EDGVC-5-08-2P_C8445.pdf" H 5900 4550 50  0001 C CNN
 F 4 "Ningbo Kangnex Elec" H 5900 4550 50  0001 C CNN "MF"
-F 5 "WJ2EDGRC-5.08-2P" H 5900 4550 50  0001 C CNN "MP"
+F 5 "WJ2EDGVC-5.08-2P" H 5900 4550 50  0001 C CNN "MP"
 F 6 "LCSC" H 5900 4550 50  0001 C CNN "Distributor"
-F 7 "C3697" H 5900 4550 50  0001 C CNN "LCSCPartN"
+F 7 "C8445" H 5900 4550 50  0001 C CNN "LCSCPartN"
 	1    5900 4550
 	1    0    0    -1

Commit message: change to vertical footprint and make some space for corrently sized courtyards
Parts:
- J106, J107, J108: footprint FootprintsTittelbach:WJ2EDGRC-5.08-2P -> FootprintsTittelbach:WJ2EDGVC-5.08-2P
Changed lines of the file:
@@
 F 0 "J106" H 5800 1350 50  0000 L CNN
 F 1 "WJ2EDGVC-5.08-2P" H 5550 1050 50  0000 L CNN
-F 2 "FootprintsTittelbach:WJ2EDGRC-5.08-2P" H 5900 1250 50  0001 C CNN
+F 2 "FootprintsTittelbach:WJ2EDGVC-5.08-2P" H 5900 1250 50  0001 C CNN
 F 3 "https://datasheet.lcsc.com/szlcsc/1912251635_Ningbo-Kangnex-Elec-WJ2EDGVC-5-08-2P_C8445.pdf" H 5900 1250 50  0001 C CNN
 F 4 "Ningbo Kangnex Elec" H 5900 1250 50  0001 C CNN "MF"
@@
 F 0 "J107" H 5800 3000 50  0000 L CNN
 F 1 "WJ2EDGVC-5.08-2P" H 5550 2700 50  0000 L CNN
-F 2 "FootprintsTittelbach:WJ2EDGRC-5.08-2P" H 5900 2900 50  0001 C CNN
+F 2 "FootprintsTittelbach:WJ2EDGVC-5.08-2P" H 5900 2900 50  0001 C CNN
 F 3 "https://datasheet.lcsc.com/szlcsc/1912251635_Ningbo-Kangnex-Elec-WJ2EDGVC-5-08-2P_C8445.pdf" H 5900 2900 50  0001 C CNN
 F 4 "Ningbo Kangnex Elec" H 5900 2900 50  0001 C CNN "MF"
@@
 F 0 "J108" H 5800 4650 50  0000 L CNN
 F 1 "WJ2EDGVC-5.08-2P" H 5550 4350 50  0000 L CNN
-F 2 "FootprintsTittelbach:WJ2EDGRC-5.08-2P" H 5900 4550 50  0001 C CNN
+F 2 "FootprintsTittelbach:WJ2EDGVC-5.08-2P" H 5900 4550 50  0001 C CNN
 F 3 "https://datasheet.lcsc.com/szlcsc/1912251635_Ningbo-Kangnex-Elec-WJ2EDGVC-5-08-2P_C8445.pdf" H 5900 4550 50  0001 C CNN
 F 4 "Ningbo Kangnex Elec" H 5900 4550 50  0001 C CNN "MF"

Commit message: update bom info and remove rescues
Parts:
- C103, C105, C106, C112, C113, C114, R107, R112, R114, R115, R116, R117, R119, R120, R121, R126, R127, R129, R130, R131, R132, R133, R134: Type (none) -> SMT
- C116: value 100P -> 100pF; Type (none) -> SMT
- D101, D102, D103: symbol lüfterklappenelektronik-rescue:D_Schottky -> Device:D_Schottky_ALT
- J106, J107, J108: Type (none) -> TH
- P101: value PWR_BUS_CONN1 -> PWR_BUS_CONN
- P109: value PWR_BUS_CONN2 -> PWR_BUS_CONN
- R101, R102, R103, R110, R111: symbol lüfterklappenelektronik-rescue:R -> Device:R
- R104, R105, R106, R109: symbol lüfterklappenelektronik-rescue:R -> Device:R; Type (none) -> SMT
- R125: value 2K -> 2K(5%)
Changed lines of the file:
@@
 $EndComp
 $Comp
-L lüfterklappenelektronik-rescue:D_Schottky D101
+L Device:D_Schottky_ALT D101
 U 1 1 57419AAE
 P 5150 1300
@@
 Connection ~ 5700 1450
 $Comp
-L lüfterklappenelektronik-rescue:R R109
+L Device:R R109
 U 1 1 57419FFE
 P 5200 1750
@@
 F 2 "Resistor_SMD:R_0603_1608Metric" V 5130 1750 50  0001 C CNN
 F 3 "" H 5200 1750 50  0000 C CNN
+F 4 "SMT" H 13550 2000 50  0001 C CNN "Type"
 	1    5200 1750
 	0    1    1    0
@@
 Connection ~ 5700 3100
 $Comp
-L lüfterklappenelektronik-rescue:R R110
+L Device:R R110
 U 1 1 5741A896
 P 5200 3400
@@
 Connection ~ 5700 4750
 $Comp
-L lüfterklappenelektronik-rescue:R R111
+L Device:R R111
 U 1 1 5741AA44
 P 5200 5050
@@
 F 2 "Resistor_SMD:R_0603_1608Metric" V 2880 6550 50  0001 C CNN
 F 3 "" H 2950 6550 50  0000 C CNN
+F 4 "SMT" V 5150 1300 50  0001 C CNN "Type"
 	1    2950 6550
 	-1   0    0    1
@@
 $EndComp
 $Comp
-L lüfterklappenelektronik-rescue:R R101
+L Device:R R101
 U 1 1 5741C2C0
 P 800 1200
@@
 $EndComp
 $Comp
-L lüfterklappenelektronik-rescue:R R102
+L Device:R R102
 U 1 1 5741D5E4
 P 800 2950
@@
 $EndComp
 $Comp
-L lüfterklappenelektronik-rescue:R R103
+L Device:R R103
 U 1 1 5741D712
 P 800 4600
@@
 F 6 "LCSC" H 8100 1150 50  0001 C CNN "Distributor"
 F 7 "C105174" H 8100 1150 50  0001 C CNN "LCSCPartN"
+F 8 "SMT" V 5150 1300 50  0001 C CNN "Type"
 	1    8100 1150
 	1    0    0    -1
@@
 F 6 "LCSC" H 8450 1150 50  0001 C CNN "Distributor"
 F 7 "C40894" H 8450 1150 50  0001 C CNN "LCSCPartN"
+F 8 "SMT" V 5150 1300 50  0001 C CNN "Type"
 	1    8450 1150
 	1    0    0    -1
@@
 P 11400 2000
 F 0 "R125" H 11470 2046 50  0000 L CNN
-F 1 "2K" H 11470 1955 50  0000 L CNN
+F 1 "2K(5%)" H 11470 1955 50  0000 L CNN
 F 2 "Resistor_SMD:R_0603_1608Metric" V 11330 2000 50  0001 C CNN
 F 3 "~" H 11400 2000 50  0001 C CNN
@@
 F 6 "LCSC" H 15100 2000 50  0001 C CNN "Distributor"
 F 7 "C42998" H 15100 2000 50  0001 C CNN "LCSCPartN"
+F 8 "SMT" V 5150 1300 50  0001 C CNN "Type"
 	1    15100 2000
 	1    0    0    -1
@@
 F 2 "Resistor_SMD:R_0603_1608Metric" V 6330 8200 50  0001 C CNN
 F 3 "~" H 6400 8200 50  0001 C CNN
+F 4 "SMT" V 5150 1300 50  0001 C CNN "Type"
 	1    6400 8200
 	1    0    0    -1
@@
 F 2 "Capacitors_SMD:C_0603" H 15438 6750 50  0001 C CNN
 F 3 "~" H 15400 6900 50  0001 C CNN
+F 4 "SMT" V 5150 1300 50  0001 C CNN "Type"
 	1    15400 6900
 	1    0    0    -1
@@
 F 2 "Resistor_SMD:R_0603_1608Metric" V 12580 7700 50  0001 C CNN
 F 3 "~" H 12650 7700 50  0001 C CNN
+F 4 "SMT" H 13550 2000 50  0001 C CNN "Type"
 	1    12650 7700
 	0    1    1    0
@@
 F 2 "Resistor_SMD:R_0603_1608Metric" V 12830 7850 50  0001 C CNN
 F 3 "~" H 12900 7850 50  0001 C CNN
+F 4 "SMT" H 13550 2000 50  0001 C CNN "Type"
 	1    12900 7850
 	1    0    0    -1
@@
 F 2 "Resistor_SMD:R_0603_1608Metric" V 15480 8350 50  0001 C CNN
 F 3 "~" H 15550 8350 50  0001 C CNN
+F 4 "SMT" V 5150 1300 50  0001 C CNN "Type"
 	1    15550 8350
 	1    0    0    -1
@@
 F 2 "Resistor_SMD:R_0603_1608Metric" V 7680 9600 50  0001 C CNN
 F 3 "~" H 7750 9600 50  0001 C CNN
+F 4 "SMT" V 5150 1300 50  0001 C CNN "Type"
 	1    7750 9600
 	0    1    1    0
@@
 F 2 "Resistor_SMD:R_0603_1608Metric" V 7680 10200 50  0001 C CNN
 F 3 "~" H 7750 10200 50  0001 C CNN
+F 4 "SMT" V 5150 1300 50  0001 C CNN "Type"
 	1    7750 10200
 	0    1    1    0
@@
 F 2 "Resistor_SMD:R_0603_1608Metric" V 3530 8350 50  0001 C CNN
 F 3 "~" H 3600 8350 50  0001 C CNN
+F 4 "SMT" V 5150 1300 50  0001 C CNN "Type"
 	1    3600 8350
 	-1   0    0    1
@@
 F 2 "Resistor_SMD:R_0603_1608Metric" V 15430 3900 50  0001 C CNN
 F 3 "~" H 15500 3900 50  0001 C CNN
+F 4 "SMT" V 5150 1300 50  0001 C CNN "Type"
 	1    15500 3900
 	0    1    1    0
@@
 F 2 "Resistor_SMD:R_0603_1608Metric" V 15430 4100 50  0001 C CNN
 F 3 "~" H 15500 4100 50  0001 C CNN
+F 4 "SMT" V 5150 1300 50  0001 C CNN "Type"
 	1    15500 4100
 	0    1    1    0
@@
 F 2 "Resistor_SMD:R_0603_1608Metric" V 10080 6350 50  0001 C CNN
 F 3 "~" H 10150 6350 50  0001 C CNN
+F 4 "SMT" V 5150 1300 50  0001 C CNN "Type"
 	1    10150 6350
 	0    1    1    0
@@
 F 2 "Resistor_SMD:R_0603_1608Metric" V 9730 6450 50  0001 C CNN
 F 3 "~" H 9800 6450 50  0001 C CNN
+F 4 "SMT" V 5150 1300 50  0001 C CNN "Type"
 	1    9800 6450
 	0    1    1    0
@@
 F 2 "Resistor_SMD:R_0603_1608Metric" V 9330 6550 50  0001 C CNN
 F 3 "~" H 9400 6550 50  0001 C CNN
+F 4 "SMT" V 5150 1300 50  0001 C CNN "Type"
 	1    9400 6550
 	0    1    1    0
@@
 P 10650 3300
 F 0 "P109" H 10569 2925 50  0000 C CNN
-F 1 "PWR_BUS_CONN2" H 10569 3016 50  0000 C CNN
+F 1 "PWR_BUS_CONN" H 10569 3016 50  0000 C CNN
 F 2 "FootprintsTittelbach:WJ2EDGRC-5.08-4P" H 10650 3300 50  0001 C CNN
 F 3 "https://datasheet.lcsc.com/szlcsc/1912251635_Ningbo-Kangnex-Elec-WJ2EDGRC-5-08-4P_C8446.pdf" H 10650 3300 50  0001 C CNN
@@
 	10150 3350 10450 3350
 $Comp
-L lüfterklappenelektronik-rescue:D_Schottky D102
+L Device:D_Schottky_ALT D102
 U 1 1 60C1928D
 P 5150 2950
@@
 $EndComp
 $Comp
-L lüfterklappenelektronik-rescue:D_Schottky D103
+L Device:D_Schottky_ALT D103
 U 1 1 60C19C0A
 P 5150 4600
@@
 F 6 "LCSC" H 7150 1150 50  0001 C CNN "Distributor"
 F 7 "C412252" H 7150 1150 50  0001 C CNN "LCSCPartN"
+F 8 "SMT" H 7150 1150 50  0001 C CNN "Type"
 	1    7150 1150
 	1    0    0    -1
@@
 F 6 "LCSC" H 14400 2000 50  0001 C CNN "Distributor"
 F 7 "C337455" H 14400 2000 50  0001 C CNN "LCSCPartN"
+F 8 "SMT" H 13550 2000 50  0001 C CNN "Type"
 	1    14400 2000
 	1    0    0    -1
@@
 F 6 "LCSC" H 5900 1250 50  0001 C CNN "Distributor"
 F 7 "C8445" H 5900 1250 50  0001 C CNN "LCSCPartN"
+F 8 "TH" H 13550 2000 50  0001 C CNN "Type"
 	1    5900 1250
 	1    0    0    -1
@@
 F 6 "LCSC" H 5900 2900 50  0001 C CNN "Distributor"
 F 7 "C8445" H 5900 2900 50  0001 C CNN "LCSCPartN"
+F 8 "TH" H 9450 3300 50  0001 C CNN "Type"
 	1    5900 2900
 	1    0    0    -1
@@
 F 6 "LCSC" H 5900 4550 50  0001 C CNN "Distributor"
 F 7 "C8445" H 5900 4550 50  0001 C CNN "LCSCPartN"
+F 8 "TH" H 13550 2000 50  0001 C CNN "Type"
 	1    5900 4550
 	1    0    0    -1
@@
 F 2 "Resistor_SMD:R_0603_1608Metric" V 5030 8700 50  0001 C CNN
 F 3 "~" H 5100 8700 50  0001 C CNN
+F 4 "SMT" V 5150 1300 50  0001 C CNN "Type"
 	1    5100 8700
 	0    1    1    0
@@
 P 800 1650
 F 0 "C116" H 915 1696 50  0000 L CNN
-F 1 "100P" H 915 1605 50  0000 L CNN
+F 1 "100pF" H 915 1605 50  0000 L CNN
 F 2 "Capacitor_SMD:C_0603_1608Metric" H 838 1500 50  0001 C CNN
 F 3 "~" H 800 1650 50  0001 C CNN
+F 4 "SMT" V 5150 1300 50  0001 C CNN "Type"
 	1    800  1650
 	1    0    0    -1
@@
 P 9450 3300
 F 0 "P101" H 9650 3250 50  0000 C CNN
-F 1 "PWR_BUS_CONN1" H 9800 3350 50  0000 C CNN
+F 1 "PWR_BUS_CONN" H 9800 3350 50  0000 C CNN
 F 2 "FootprintsTittelbach:WJ2EDGRC-5.08-4P" H 9450 3300 50  0001 C CNN
 F 3 "https://datasheet.lcsc.com/szlcsc/1912251635_Ningbo-Kangnex-Elec-WJ2EDGRC-5-08-4P_C8446.pdf" H 9450 3300 50  0001 C CNN
@@
 F 2 "Resistor_SMD:R_0603_1608Metric" V 9130 7350 50  0001 C CNN
 F 3 "~" H 9200 7350 50  0001 C CNN
+F 4 "SMT" V 5150 1300 50  0001 C CNN "Type"
 	1    9200 7350
 	1    0    0    -1
@@
 F 2 "Resistor_SMD:R_0603_1608Metric" V 3130 4650 50  0001 C CNN
 F 3 "~" H 3200 4650 50  0001 C CNN
+F 4 "SMT" H 13550 2000 50  0001 C CNN "Type"
 	1    3200 4650
 	1    0    0    -1
@@
 F 2 "Resistor_SMD:R_0603_1608Metric" V 3130 3000 50  0001 C CNN
 F 3 "~" H 3200 3000 50  0001 C CNN
+F 4 "SMT" H 13550 2000 50  0001 C CNN "Type"
 	1    3200 3000
 	1    0    0    -1
@@
 EndstopDamper3
 $Comp
-L lüfterklappenelektronik-rescue:R R106
+L Device:R R106
 U 1 1 5741D727
 P 3500 4900
@@
 F 2 "Resistor_SMD:R_0603_1608Metric" V 3430 4900 50  0001 C CNN
 F 3 "" H 3500 4900 50  0000 C CNN
+F 4 "SMT" H 13550 2000 50  0001 C CNN "Type"
 	1    3500 4900
 	0    1    1    0
@@
 EndstopDamper2
 $Comp
-L lüfterklappenelektronik-rescue:R R105
+L Device:R R105
 U 1 1 5741D5F9
 P 3500 3250
@@
 F 2 "Resistor_SMD:R_0603_1608Metric" V 3430 3250 50  0001 C CNN
 F 3 "" H 3500 3250 50  0000 C CNN
+F 4 "SMT" H 13550 2000 50  0001 C CNN "Type"
 	1    3500 3250
 	0    1    1    0
@@
 EndstopDamper1
 $Comp
-L lüfterklappenelektronik-rescue:R R104
+L Device:R R104
 U 1 1 5741CC61
 P 3400 1500
@@
 F 2 "Resistor_SMD:R_0603_1608Metric" V 3330 1500 50  0001 C CNN
 F 3 "" H 3400 1500 50  0000 C CNN
+F 4 "SMT" H 13550 2000 50  0001 C CNN "Type"
 	1    3400 1500
 	0    1    1    0
